Commit message: Added EKF - visualize condition

File: scout_mini_description/models/scout_mini/xacro/scout_mini.xacro (robot description, xacro)
@@ -52,7 +52,11 @@
         <child link="inertial_link" />
     </joint>
+    <link name="base_footprint" />
+    <joint name="base_footprint_joint" type="fixed">
+        <origin xyz="0 0 -0.16" />
+        <parent link="base_link"/>
+        <child link="base_footprint"/>
+    </joint>
     <!-- Scout wheel macros -->
-    <!-- wheel labeled from 0 to 3, conter-clockwise, starting from front right wheel -->
-    <!-- motor 1 and 2 (left side) are mechanically installed in a reversed direction -->
     <xacro:scout_mini_wheel wheel_prefix="front_right" >
         <origin xyz= "0 0 0" rpy="1.57 0 0" />
@@ -84,5 +88,3 @@
         <child link="rear_mount" />
     </joint>
-    <!-- Gazebo definitions  -->
-    <!-- <xacro:include filename="$(find scout_description)/urdf/scout_mini.gazebo" /> -->
 </robot>
