Commit message: Updated EKF Node

File: scout_mini_description/models/scout_mini/xacro/scout_mini_viz.xacro (robot description, xacro)
@@ -1,14 +1,69 @@
 <?xml version="1.0"?>
-<robot name="zed_cameras" xmlns:xacro="http://www.ros.org/wiki/xacro">
-    <xacro:include filename="$(find zed_wrapper)/urdf/zed_macro.urdf.xacro" />
-    <xacro:include filename="$(find scout_mini_description)/models/scout_mini/xacro/scout_mini.xacro" />
-    <joint name="zed_mount_joint" type="fixed">
-        <origin xyz="0.277812 0 0.108212" rpy="0 0 0" />
-        <parent link="commander_slim_link" />
-        <child link="zed_mount_link" />
+<robot name="scout_mini" xmlns:xacro="http://ros.org/wiki/xacro">
+    <xacro:include
+        filename="$(find scout_mini_description)/models/scout_mini/xacro/scout_mini_wheel.xacro" />
+    <xacro:include
+        filename="$(find scout_mini_description)/models/commander_slim/xacro/commander_slim.xacro" />
+       <xacro:property name="M_PI" value="3.14159" />
+    <!-- Vehicle Geometries -->
+    <xacro:property name="base_x_size" value="0.6200000" />
+    <xacro:property name="base_y_size" value="0.585000" />
+    <xacro:property name="base_z_size" value="0.235000" />
+    <xacro:property name="wheelbase" value="0.463951" />
+    <xacro:property name="track" value="0.416503" />
+    <xacro:property name="wheel_vertical_offset" value="-0.100998" />
+    <xacro:property name="wheel_length" value="0.8e-01" />
+    <xacro:property name="wheel_radius" value="1.600e-01" />
+    <xacro:property name="robot_namespace" value="/scout_mini" />
+    <!-- Base link -->
+    <link name="base_link">
+        <visual>
+            <origin
+                xyz="0 0 0"
+                rpy="1.5707 0 -1.5707" />
+            <geometry>
+                <mesh
+                    filename="package://scout_mini_description/models/scout_mini/meshes/scout_mini_base_link.dae" />
+            </geometry>
+        </visual>
+        <collision>
+            <origin
+                xyz="0 0 0"
+                rpy="1.5707 0 -1.5707" />
+            <geometry>
+                <mesh
+                    filename="package://scout_mini_description/models/scout_mini/meshes/scout_mini_base_link.dae" />
+            </geometry>
+        </collision>
+    </link>
+    <link name="inertial_link">
+        <inertial>
+            <mass value="60" />
+            <origin xyz="0.0 0.0 0.0" />
+            <inertia ixx="2.288641" ixy="0" ixz="0" iyy="5.103976" iyz="0" izz="3.431465" />
+        </inertial>
+    </link>
+    <joint name="inertial_joint" type="fixed">
+        <origin xyz="0 0 0" rpy="0 0 0" />
+        <parent link="base_link" />
+        <child link="inertial_link" />
     </joint>
-    <link name="zed_mount_link" />
-    <xacro:zed_camera name="zed2" model="zed2" parent="zed_mount_link">
-        <origin xyz="0 0 0" rpy="0 0 0" />
-    </xacro:zed_camera>
+    <link name="base_footprint" />
+    <joint name="base_footprint_joint" type="fixed">
+        <origin xyz="0 0 -0.16" />
+        <parent link="base_link"/>
+        <child link="base_footprint"/>
+    </joint>
+    <link name="front_mount" />
+    <joint name="front_mount_joint" type="fixed">
+        <origin xyz="0.175 0 0.068999" rpy="0 0 0" />
+        <parent link="base_link" />
+        <child link="front_mount" />
+    </joint>
+    <link name="rear_mount" />
+    <joint name="rear_mount_joint" type="fixed">
+        <origin xyz="-0.175 0 0.068999" rpy="0 0 0" />
+        <parent link="base_link" />
+        <child link="rear_mount" />
+    </joint>
 </robot>

File: scout_mini_description/models/scout_mini/xacro/scout_mini_wheel.xacro (robot description, xacro)
@@ -23,5 +23,5 @@
             </collision>
         </link>
-        <joint name="${wheel_prefix}_wheel" type="continuous">
+        <joint name="${wheel_prefix}_wheel" type="fixed">
             <parent link="base_link" />
             <child link="${wheel_prefix}_wheel_link" />
