Commit message: Added EKF - visualize condition

File: scout_mini_description/models/scout_mini/xacro/scout_mini_wheel.xacro (robot description, xacro)
@@ -10,5 +10,4 @@
             <visual>
                 <xacro:insert_block name="visual_origin" />
-                <!-- <origin xyz="0 0 0" rpy="0 0 ${rotation}" /> -->
                 <geometry>
                     <mesh
@@ -18,7 +17,4 @@
             <collision>
                 <xacro:insert_block name="visual_origin" />
-                <!-- <origin
-                    xyz="0 0 0"
-                    rpy="0 0 ${rotation}" /> -->
                 <geometry>
                     <mesh
@@ -27,6 +23,5 @@
             </collision>
         </link>
-        <joint name="${wheel_prefix}_wheel" type="continuous"> <!-- MAKE SURE TO SET THIS BACK TO
-            CONTINUOUS ONCE THE JOINTS ARE PUBLISHED -->
+        <joint name="${wheel_prefix}_wheel" type="continuous">
             <parent link="base_link" />
             <child link="${wheel_prefix}_wheel_link" />

Commit message: Working simulated odometry and EKF Node

File: scout_mini_description/models/scout_mini/xacro/scout_mini_wheel.xacro (robot description, xacro)
@@ -1,5 +1,5 @@
 <?xml version="1.0"?>
 <robot xmlns:xacro="http://ros.org/wiki/xacro" name="scout_wheel">
-    <xacro:macro name="scout_mini_wheel" params="wheel_prefix joint_type *visual_origin *joint_pose">
+    <xacro:macro name="scout_mini_wheel" params="wheel_prefix *visual_origin *joint_pose">
         <link name="${wheel_prefix}_wheel_link">
             <inertial>
@@ -23,5 +23,5 @@
             </collision>
         </link>
-        <joint name="${wheel_prefix}_wheel" type="${joint_type}">
+        <joint name="${wheel_prefix}_wheel" type="continuous">
             <parent link="base_link" />
             <child link="${wheel_prefix}_wheel_link" />

File: scout_mini_gazebo/models/scout_mini/xacro/scout_mini.xacro (robot description, xacro)
@@ -6,5 +6,7 @@
         filename="$(find scout_mini_description)/models/commander_slim/xacro/commander_slim.xacro" />
     <xacro:include
-        filename="$(find scout_mini_description)/models/scout_mini/xacro/scout_mini_gazebo.xacro" />
+        filename="$(find scout_mini_gazebo)/models/scout_mini/xacro/scout_mini_gazebo.xacro" />
+    <xacro:include
+        filename="$(find scout_mini_gazebo)/models/scout_mini/xacro/scout_mini_sensors.xacro" />
     <xacro:property name="M_PI" value="3.14159" />
     <!-- Vehicle Geometries -->
@@ -51,31 +53,33 @@
         <child link="inertial_link" />
     </joint>
-        <!-- Scout wheel macros -->
-    <xacro:scout_mini_wheel wheel_prefix="front_right" joint_type="continuous" >
-        <origin xyz= "0 0 0" rpy="1.57 0 0" />
+    <!-- Scout wheel macros -->
+    <xacro:scout_mini_wheel wheel_prefix="front_right">
+        <origin xyz="0 0 0" rpy="1.57 0 0" />
         <origin xyz="${wheelbase/2} ${-track/2} ${wheel_vertical_offset}" rpy="0 0 0" />
     </xacro:scout_mini_wheel>
-    <xacro:scout_mini_wheel wheel_prefix="front_left" joint_type="continuous" >
-        <origin xyz= "0 0 0" rpy="-1.57 0 0" />
+    <xacro:scout_mini_wheel wheel_prefix="front_left">
+        <origin xyz="0 0 0" rpy="-1.57 0 0" />
         <origin xyz="${wheelbase/2} ${track/2} ${wheel_vertical_offset}" rpy="0 0 0" />
     </xacro:scout_mini_wheel>
-    <xacro:scout_mini_wheel wheel_prefix="rear_left" joint_type="continuous" >
-        <origin xyz= "0 0 0" rpy="-1.57 0 0" />
+    <xacro:scout_mini_wheel wheel_prefix="rear_left">
+        <origin xyz="0 0 0" rpy="-1.57 0 0" />
         <origin xyz="${-wheelbase/2} ${track/2} ${wheel_vertical_offset}" rpy="0 0 0" />
     </xacro:scout_mini_wheel>
-    <xacro:scout_mini_wheel wheel_prefix="rear_right" joint_type="continuous" >
-        <origin xyz= "0 0 0" rpy="1.57 0 0" />
+    <xacro:scout_mini_wheel wheel_prefix="rear_right">
+        <origin xyz="0 0 0" rpy="1.57 0 0" />
         <origin xyz="${-wheelbase/2} ${-track/2} ${wheel_vertical_offset}" rpy="0 0 0" />
     </xacro:scout_mini_wheel>
     <xacro:diff_drive_plugin />
+    <xacro:IMU />
+    <xacro:depth_camera />
     <link name="base_footprint" />
     <joint name="base_footprint_joint" type="fixed">
-        <origin xyz="0 0 -0.16" />
-        <parent link="base_footprint"/>
-        <child link="base_link"/>
+        <origin xyz="0 0 0.16" />
+        <parent link="base_footprint" />
+        <child link="base_link" />
     </joint>
     <link name="front_mount" />
     <joint name="front_mount_joint" type="fixed">
-        <origin xyz="0.175 0 0.068999" rpy="0 0 0" />
+        <origin xyz="0.175 0 0.068999" rpy  ="0 0 0" />
         <parent link="base_link" />
         <child link="front_mount" />

File: scout_mini_gazebo/models/scout_mini/xacro/scout_mini_gazebo.xacro (robot description, xacro)
@@ -6,4 +6,5 @@
                 <ros>
                     <namespace>${robot_namespace}</namespace>
+                    <remapping>odom:=zed_node/odom</remapping>
                 </ros>
                 <!-- Update rate in Hz -->
@@ -26,10 +27,10 @@
                 <command_topic>cmd_vel</command_topic>
                 <!-- output -->
-                <publish_odom>false</publish_odom>
+                <publish_odom>true</publish_odom>
                 <publish_odom_tf>false</publish_odom_tf>
                 <publish_wheel_tf>true</publish_wheel_tf>
-                <odometry_topic>odom</odometry_topic>
+                <odometry_topic>zed_node/odom</odometry_topic>
                 <odometry_frame>odom</odometry_frame>
-                <robot_base_frame>base_link</robot_base_frame>
+                <robot_base_frame>base_footprint</robot_base_frame>
             </plugin>
         </gazebo>

File: scout_mini_gazebo/models/scout_mini/xacro/scout_mini_sensors.xacro (robot description, xacro)
@@ -2,5 +2,5 @@
 <robot name="scout_mini_sensors" xmlns:xacro="http://wiki.ros.org/xacro">
     <xacro:include filename="$(find zed_wrapper)/urdf/zed_macro.urdf.xacro" />
-    <xacro:macro name="zed_cameras">
+    <xacro:macro name="depth_camera">
         <joint name="zed_mount_joint" type="fixed">
             <origin xyz="0.277812 0 0.108212" rpy="0 0 0" />
@@ -9,9 +9,181 @@
         </joint>
         <link name="zed_mount_link" />
-        <xacro:zed_camera name="zed2" model="zed2" parents="zed_mount_link">
+        <xacro:zed_camera name="zed2" model="zed2" parent="zed_mount_link">
             <origin xyz="0 0 0" rpy="0 0 0" />
         </xacro:zed_camera>
         <link name="zed_depth_link_optical" />
-        <joint name="zed_depth_joint_
+        <joint name="zed_depth_join_optical" type="fixed">
+            <parent link="zed_mount_link" />
+            <child link="zed_depth_link_optical" />
+            <origin xyz="0 0 0" rpy="${-pi/2} 0 ${-pi/2}" />
+        </joint>
+        <gazebo reference="zed_mount_link">
+            <sensor type="depth" name="zed_depth_camera">
+                <visualize>false</visualize>
+                <update_rate>10.0</update_rate>
+                <always_on>true</always_on>
+                <pose>0 0 0 0 0 0</pose>
+                <camera name="zed_depth_camera">
+                    <horizontal_fov>1.91986</horizontal_fov>
+                    <vertical_fov>1.22173</vertical_fov>
+                    <image>
+                        <width>1344</width>
+                        <height>376</height>
+                        <format>B8G8R8</format>
+                    </image>
+                    <clip>
+                        <near>0.2</near>
+                        <far>20</far>
+                    </clip>
+                </camera>
+                <plugin name="zed_camera_depth_controller" filename="libgazebo_ros_camera.so">
+                    <ros>
+                        <namespace>${robot_namespace}</namespace>
+                        <!-- Remappings for the ZED Camera Nodes -->
+                    </ros>
+                    <frame_name>zed_depth_link_optical</frame_name>
+                    <cameraName>zed_depth_camera</cameraName>
+                    <hack_baseline>0.07</hack_baseline>
+                    <min_depth>0.2</min_depth>
+                    <max_depth>20</max_depth>
+                </plugin>
+            </sensor>
+            <sensor name="ZED_IMU_sensor" type="imu">
+                <plugin filename="libgazebo_ros_imu_sensor.so" name="ZED_IMU_plugin">
+                    <ros>
+                        <namespace>${robot_namespace}</namespace>
+                        <remapping>~/out:=zed_node/imu/data</remapping>
+                    </ros>
+                    <initial_orientation_as_reference>false</initial_orientation_as_reference>
+                </plugin>
+                <always_on>true</always_on>
+                <update_rate>100</update_rate>
+                <visualize>true</visualize>
+                <!-- <imu>
+                    <angular_velocity>
+                        <x>
+                            <noise type="gaussian">
+                                <mean>0.0</mean>
+                                <stddev>2e-4</stddev>
+                                <bias_mean>0.0000075</bias_mean>
+                                <bias_stddev>0.0000008</bias_stddev>
+                            </noise>
+                        </x>
+                        <y>
+                            <noise type="gaussian">
+                                <mean>0.0</mean>
+                                <stddev>2e-4</stddev>
+                                <bias_mean>0.0000075</bias_mean>
+                                <bias_stddev>0.0000008</bias_stddev>
+                            </noise>
+                        </y>
+                        <z>
+                            <noise type="gaussian">
+                                <mean>0.0</mean>
+                                <stddev>2e-4</stddev>
+                                <bias_mean>0.0000075</bias_mean>
+                                <bias_stddev>0.0000008</bias_stddev>
+                            </noise>
+                        </z>
+                    </angular_velocity>
+                    <linear_acceleration>
+                        <x>
+                            <noise type="gaussian">
+                                <mean>0.0</mean>
+                                <stddev>1.7e-2</stddev>
+                                <bias_mean>0.1</bias_mean>
+                                <bias_stddev>0.001</bias_stddev>
+                            </noise>
+                        </x>
+                        <y>
+                            <noise type="gaussian">
+                                <mean>0.0</mean>
+                                <stddev>1.7e-2</stddev>
+                                <bias_mean>0.1</bias_mean>
+                                <bias_stddev>0.001</bias_stddev>
+                            </noise>
+                        </y>
+                        <z>
+                            <noise type="gaussian">
+                                <mean>0.0</mean>
+                                <stddev>1.7e-2</stddev>
+                                <bias_mean>0.1</bias_mean>
+                                <bias_stddev>0.001</bias_stddev>
+                            </noise>
+                        </z>
+                    </linear_acceleration>
+                </imu> -->
+            </sensor>
+        </gazebo>
+    </xacro:macro>
+    <xacro:macro name="IMU">
+        <gazebo reference="IMU">
+            <sensor name="IMU_sensor" type="imu">
+                <plugin filename="libgazebo_ros_imu_sensor.so" name="IMU_plugin">
+                    <ros>
+                        <namespace>${robot_namespace}</namespace>
+                        <remapping>~/out:=imu/data</remapping>
+                    </ros>
+                    <initial_orientation_as_reference>false</initial_orientation_as_reference>
+                </plugin>
+                <always_on>true</always_on>
+                <update_rate>100</update_rate>
+                <visualize>true</visualize>
+                <imu>
+                    <angular_velocity>
+                        <x>
+                            <noise type="gaussian">
+                                <mean>0.0</mean>
+                                <stddev>2e-4</stddev>
+                                <bias_mean>0.0000075</bias_mean>
+                                <bias_stddev>0.0000008</bias_stddev>
+                            </noise>
+                        </x>
+                        <y>
+                            <noise type="gaussian">
+                                <mean>0.0</mean>
+                                <stddev>2e-4</stddev>
+                                <bias_mean>0.0000075</bias_mean>
+                                <bias_stddev>0.0000008</bias_stddev>
+                            </noise>
+                        </y>
+                        <z>
+                            <noise type="gaussian">
+                                <mean>0.0</mean>
+                                <stddev>2e-4</stddev>
+                                <bias_mean>0.0000075</bias_mean>
+                                <bias_stddev>0.0000008</bias_stddev>
+                            </noise>
+                        </z>
+                    </angular_velocity>
+                    <linear_acceleration>
+                        <x>
+                            <noise type="gaussian">
+                                <mean>0.0</mean>
+                                <stddev>1.7e-2</stddev>
+                                <bias_mean>0.1</bias_mean>
+                                <bias_stddev>0.001</bias_stddev>
+                            </noise>
+                        </x>
+                        <y>
+                            <noise type="gaussian">
+                                <mean>0.0</mean>
+                                <stddev>1.7e-2</stddev>
+                                <bias_mean>0.1</bias_mean>
+                                <bias_stddev>0.001</bias_stddev>
+                            </noise>
+                        </y>
+                        <z>
+                            <noise type="gaussian">
+                                <mean>0.0</mean>
+                                <stddev>1.7e-2</stddev>
+                                <bias_mean>0.1</bias_mean>
+                                <bias_stddev>0.001</bias_stddev>
+                            </noise>
+                        </z>
+                    </linear_acceleration>
+                </imu>
+            </sensor>
+        </gazebo>
     </xacro:macro>
 </robot>
