Commit message: nav2 launch setup - fixed TF

File: scout_mini_description/models/scout_mini/xacro/scout_mini_tf.xacro (robot description, xacro)
@@ -3,6 +3,4 @@
     <xacro:include
         filename="$(find scout_mini_description)/models/scout_mini/xacro/scout_mini_wheel.xacro" />
-    <xacro:include
-        filename="$(find scout_mini_description)/models/scout_mini/xacro/scout_mini_gazebo.xacro" />
     <xacro:include
         filename="$(find scout_mini_description)/models/commander_slim/xacro/commander_slim.xacro" />
@@ -59,21 +57,20 @@
     </joint>
     <!-- Scout wheel macros -->
-    <xacro:scout_mini_wheel wheel_prefix="front_right" >
+    <xacro:scout_mini_wheel wheel_prefix="front_right" joint_type="fixed" >
         <origin xyz= "0 0 0" rpy="1.57 0 0" />
         <origin xyz="${wheelbase/2} ${-track/2} ${wheel_vertical_offset}" rpy="0 0 0" />
     </xacro:scout_mini_wheel>
-    <xacro:scout_mini_wheel wheel_prefix="front_left" >
+    <xacro:scout_mini_wheel wheel_prefix="front_left" joint_type="fixed" >
         <origin xyz= "0 0 0" rpy="-1.57 0 0" />
         <origin xyz="${wheelbase/2} ${track/2} ${wheel_vertical_offset}" rpy="0 0 0" />
     </xacro:scout_mini_wheel>
-    <xacro:scout_mini_wheel wheel_prefix="rear_left" >
+    <xacro:scout_mini_wheel wheel_prefix="rear_left" joint_type="fixed" >
         <origin xyz= "0 0 0" rpy="-1.57 0 0" />
         <origin xyz="${-wheelbase/2} ${track/2} ${wheel_vertical_offset}" rpy="0 0 0" />
     </xacro:scout_mini_wheel>
-    <xacro:scout_mini_wheel wheel_prefix="rear_right" >
+    <xacro:scout_mini_wheel wheel_prefix="rear_right" joint_type="fixed" >
         <origin xyz= "0 0 0" rpy="1.57 0 0" />
         <origin xyz="${-wheelbase/2} ${-track/2} ${wheel_vertical_offset}" rpy="0 0 0" />
     </xacro:scout_mini_wheel>
-    <xacro:diff_drive_plugin />
     <link name="front_mount" />
     <joint name="front_mount_joint" type="fixed">

File: scout_mini_description/models/scout_mini/xacro/scout_mini_viz.xacro (robot description, xacro)
@@ -5,5 +5,7 @@
     <xacro:include
         filename="$(find scout_mini_description)/models/commander_slim/xacro/commander_slim.xacro" />
-       <xacro:property name="M_PI" value="3.14159" />
+    <xacro:include
+        filename="$(find scout_mini_description)/models/scout_mini/xacro/scout_mini_gazebo.xacro" />
+    <xacro:property name="M_PI" value="3.14159" />
     <!-- Vehicle Geometries -->
     <xacro:property name="base_x_size" value="0.6200000" />
@@ -49,9 +51,27 @@
         <child link="inertial_link" />
     </joint>
+        <!-- Scout wheel macros -->
+    <xacro:scout_mini_wheel wheel_prefix="front_right" joint_type="continuous" >
+        <origin xyz= "0 0 0" rpy="1.57 0 0" />
+        <origin xyz="${wheelbase/2} ${-track/2} ${wheel_vertical_offset}" rpy="0 0 0" />
+    </xacro:scout_mini_wheel>
+    <xacro:scout_mini_wheel wheel_prefix="front_left" joint_type="continuous" >
+        <origin xyz= "0 0 0" rpy="-1.57 0 0" />
+        <origin xyz="${wheelbase/2} ${track/2} ${wheel_vertical_offset}" rpy="0 0 0" />
+    </xacro:scout_mini_wheel>
+    <xacro:scout_mini_wheel wheel_prefix="rear_left" joint_type="continuous" >
+        <origin xyz= "0 0 0" rpy="-1.57 0 0" />
+        <origin xyz="${-wheelbase/2} ${track/2} ${wheel_vertical_offset}" rpy="0 0 0" />
+    </xacro:scout_mini_wheel>
+    <xacro:scout_mini_wheel wheel_prefix="rear_right" joint_type="continuous" >
+        <origin xyz= "0 0 0" rpy="1.57 0 0" />
+        <origin xyz="${-wheelbase/2} ${-track/2} ${wheel_vertical_offset}" rpy="0 0 0" />
+    </xacro:scout_mini_wheel>
+    <xacro:diff_drive_plugin />
     <link name="base_footprint" />
     <joint name="base_footprint_joint" type="fixed">
         <origin xyz="0 0 -0.16" />
-        <parent link="base_link"/>
-        <child link="base_footprint"/>
+        <parent link="base_footprint"/>
+        <child link="base_link"/>
     </joint>
     <link name="front_mount" />

File: scout_mini_description/models/scout_mini/xacro/scout_mini_wheel.xacro (robot description, xacro)
@@ -1,5 +1,5 @@
 <?xml version="1.0"?>
 <robot xmlns:xacro="http://ros.org/wiki/xacro" name="scout_wheel">
-    <xacro:macro name="scout_mini_wheel" params="wheel_prefix *visual_origin *joint_pose">
+    <xacro:macro name="scout_mini_wheel" params="wheel_prefix joint_type *visual_origin *joint_pose">
         <link name="${wheel_prefix}_wheel_link">
             <inertial>
@@ -23,5 +23,5 @@
             </collision>
         </link>
-        <joint name="${wheel_prefix}_wheel" type="fixed">
+        <joint name="${wheel_prefix}_wheel" type="${joint_type}">
             <parent link="base_link" />
             <child link="${wheel_prefix}_wheel_link" />

Commit message: Working depth_image_to_laserscan

File: scout_mini_description/models/scout_mini/xacro/scout_mini_tf.xacro (robot description, xacro)
@@ -53,6 +53,6 @@
     <joint name="base_footprint_joint" type="fixed">
         <origin xyz="0 0 -0.16" />
-        <parent link="base_link"/>
-        <child link="base_footprint"/>
+        <parent link="base_footprint"/>
+        <child link="base_link"/>
     </joint>
     <!-- Scout wheel macros -->

File: scout_mini_description/models/scout_mini/xacro/scout_mini_wheel.xacro (robot description, xacro)
@@ -1,5 +1,5 @@
 <?xml version="1.0"?>
 <robot xmlns:xacro="http://ros.org/wiki/xacro" name="scout_wheel">
-    <xacro:macro name="scout_mini_wheel" params="wheel_prefix *visual_origin *joint_pose">
+    <xacro:macro name="scout_mini_wheel" params="wheel_prefix joint_type *visual_origin *joint_pose">
         <link name="${wheel_prefix}_wheel_link">
             <inertial>
@@ -23,5 +23,5 @@
             </collision>
         </link>
-        <joint name="${wheel_prefix}_wheel" type="continuous">
+        <joint name="${wheel_prefix}_wheel" type="${joint_type}">
             <parent link="base_link" />
             <child link="${wheel_prefix}_wheel_link" />

File: scout_mini_gazebo/models/scout_mini/xacro/scout_mini.xacro (robot description, xacro)
@@ -54,17 +54,17 @@
     </joint>
     <!-- Scout wheel macros -->
-    <xacro:scout_mini_wheel wheel_prefix="front_right">
+    <xacro:scout_mini_wheel wheel_prefix="front_right" joint_type="continuous">
         <origin xyz="0 0 0" rpy="1.57 0 0" />
         <origin xyz="${wheelbase/2} ${-track/2} ${wheel_vertical_offset}" rpy="0 0 0" />
     </xacro:scout_mini_wheel>
-    <xacro:scout_mini_wheel wheel_prefix="front_left">
+    <xacro:scout_mini_wheel wheel_prefix="front_left" joint_type="continuous">
         <origin xyz="0 0 0" rpy="-1.57 0 0" />
         <origin xyz="${wheelbase/2} ${track/2} ${wheel_vertical_offset}" rpy="0 0 0" />
     </xacro:scout_mini_wheel>
-    <xacro:scout_mini_wheel wheel_prefix="rear_left">
+    <xacro:scout_mini_wheel wheel_prefix="rear_left" joint_type="continuous">
         <origin xyz="0 0 0" rpy="-1.57 0 0" />
         <origin xyz="${-wheelbase/2} ${track/2} ${wheel_vertical_offset}" rpy="0 0 0" />
     </xacro:scout_mini_wheel>
-    <xacro:scout_mini_wheel wheel_prefix="rear_right">
+    <xacro:scout_mini_wheel wheel_prefix="rear_right" joint_type="continuous">
         <origin xyz="0 0 0" rpy="1.57 0 0" />
         <origin xyz="${-wheelbase/2} ${-track/2} ${wheel_vertical_offset}" rpy="0 0 0" />

File: scout_mini_gazebo/models/scout_mini/xacro/scout_mini_gazebo.xacro (robot description, xacro)
@@ -9,5 +9,5 @@
                 </ros>
                 <!-- Update rate in Hz -->
-                <update_rate>50</update_rate>
+                <update_rate>30</update_rate>
                 <!-- wheels -->
                 <num_wheel_pairs>2</num_wheel_pairs>
@@ -32,5 +32,5 @@
                 <odometry_topic>zed_node/odom</odometry_topic>
                 <odometry_frame>odom</odometry_frame>
-                <robot_base_frame>base_link</robot_base_frame>
+                <robot_base_frame>base_footprint</robot_base_frame>
             </plugin>
         </gazebo>

File: scout_mini_gazebo/models/scout_mini/xacro/scout_mini_sensors.xacro (robot description, xacro)
@@ -12,14 +12,8 @@
             <origin xyz="0 0 0" rpy="0 0 0" />
         </xacro:zed_camera>
-        <link name="zed_depth_link_optical" />
-        <joint name="zed_depth_joint_optical" type="fixed">
-            <parent link="zed_mount_link" />
-            <child link="zed_depth_link_optical" />
-            <origin xyz="0 0 0" rpy="${-pi/2} 0 ${-pi/2}" />
-        </joint>
         <gazebo reference="zed2_camera_center">
             <sensor type="depth" name="zed_depth_camera">
                 <visualize>false</visualize>
-                <update_rate>10.0</update_rate>
+                <update_rate>30.0</update_rate>
                 <always_on>true</always_on>
                 <pose>0 0 0 0 0 0</pose>

Commit message: NAV2 Bringup functioning - Gazebo fix

File: scout_mini_description/models/scout_mini/xacro/scout_mini_tf.xacro (robot description, xacro)
@@ -57,17 +57,17 @@
     </joint>
     <!-- Scout wheel macros -->
-    <xacro:scout_mini_wheel wheel_prefix="front_right" joint_type="fixed" >
+    <xacro:scout_mini_wheel wheel_prefix="front_right" joint_type="fixed" reflect="-1">
         <origin xyz= "0 0 0" rpy="1.57 0 0" />
         <origin xyz="${wheelbase/2} ${-track/2} ${wheel_vertical_offset}" rpy="0 0 0" />
     </xacro:scout_mini_wheel>
-    <xacro:scout_mini_wheel wheel_prefix="front_left" joint_type="fixed" >
+    <xacro:scout_mini_wheel wheel_prefix="front_left" joint_type="fixed" reflect="1">
         <origin xyz= "0 0 0" rpy="-1.57 0 0" />
         <origin xyz="${wheelbase/2} ${track/2} ${wheel_vertical_offset}" rpy="0 0 0" />
     </xacro:scout_mini_wheel>
-    <xacro:scout_mini_wheel wheel_prefix="rear_left" joint_type="fixed" >
+    <xacro:scout_mini_wheel wheel_prefix="rear_left" joint_type="fixed" reflect="1">
         <origin xyz= "0 0 0" rpy="-1.57 0 0" />
         <origin xyz="${-wheelbase/2} ${track/2} ${wheel_vertical_offset}" rpy="0 0 0" />
     </xacro:scout_mini_wheel>
-    <xacro:scout_mini_wheel wheel_prefix="rear_right" joint_type="fixed" >
+    <xacro:scout_mini_wheel wheel_prefix="rear_right" joint_type="fixed" reflect="-1">
         <origin xyz= "0 0 0" rpy="1.57 0 0" />
         <origin xyz="${-wheelbase/2} ${-track/2} ${wheel_vertical_offset}" rpy="0 0 0" />

File: scout_mini_description/models/scout_mini/xacro/scout_mini_wheel.xacro (robot description, xacro)
@@ -1,10 +1,10 @@
 <?xml version="1.0"?>
 <robot xmlns:xacro="http://ros.org/wiki/xacro" name="scout_wheel">
-    <xacro:macro name="scout_mini_wheel" params="wheel_prefix joint_type *visual_origin *joint_pose">
+    <xacro:macro name="scout_mini_wheel" params="reflect wheel_prefix joint_type *visual_origin *joint_pose">
         <link name="${wheel_prefix}_wheel_link">
             <inertial>
                 <mass value="3" />
-                <origin xyz="0 0 0" />
-                <inertia ixx="0.7171" ixy="0" ixz="0" iyy="0.7171" iyz="0" izz="0.1361" />
+                <origin xyz="0 ${reflect * 0.05} 0" />
+                <inertia ixx="0.012" ixy="0" ixz="0" iyy="0.012" iyz="0" izz="0.012" />
             </inertial>
             <visual>

File: scout_mini_gazebo/models/scout_mini/xacro/scout_mini.xacro (robot description, xacro)
@@ -45,5 +45,6 @@
             <mass value="60" />
             <origin xyz="0.0 0.0 0.0" />
-            <inertia ixx="2.288641" ixy="0" ixz="0" iyy="5.103976" iyz="0" izz="3.431465" />
+            <!-- <inertia ixx="2.288641" ixy="0" ixz="0" iyy="5.103976" iyz="0" izz="3.431465" /> -->
+            <inertia ixx="3.0" ixy="0" ixz="0" iyy="3.0" iyz="0" izz="3.431465" />
         </inertial>
     </link>
@@ -54,17 +55,17 @@
     </joint>
     <!-- Scout wheel macros -->
-    <xacro:scout_mini_wheel wheel_prefix="front_right" joint_type="continuous">
+    <xacro:scout_mini_wheel wheel_prefix="front_right" joint_type="continuous" reflect="-1">
         <origin xyz="0 0 0" rpy="1.57 0 0" />
         <origin xyz="${wheelbase/2} ${-track/2} ${wheel_vertical_offset}" rpy="0 0 0" />
     </xacro:scout_mini_wheel>
-    <xacro:scout_mini_wheel wheel_prefix="front_left" joint_type="continuous">
+    <xacro:scout_mini_wheel wheel_prefix="front_left" joint_type="continuous" reflect="1">
         <origin xyz="0 0 0" rpy="-1.57 0 0" />
         <origin xyz="${wheelbase/2} ${track/2} ${wheel_vertical_offset}" rpy="0 0 0" />
     </xacro:scout_mini_wheel>
-    <xacro:scout_mini_wheel wheel_prefix="rear_left" joint_type="continuous">
+    <xacro:scout_mini_wheel wheel_prefix="rear_left" joint_type="continuous" reflect="1">
         <origin xyz="0 0 0" rpy="-1.57 0 0" />
         <origin xyz="${-wheelbase/2} ${track/2} ${wheel_vertical_offset}" rpy="0 0 0" />
     </xacro:scout_mini_wheel>
-    <xacro:scout_mini_wheel wheel_prefix="rear_right" joint_type="continuous">
+    <xacro:scout_mini_wheel wheel_prefix="rear_right" joint_type="continuous" reflect="-1">
         <origin xyz="0 0 0" rpy="1.57 0 0" />
         <origin xyz="${-wheelbase/2} ${-track/2} ${wheel_vertical_offset}" rpy="0 0 0" />

File: scout_mini_gazebo/models/scout_mini/xacro/scout_mini_gazebo.xacro (robot description, xacro)
@@ -35,4 +35,48 @@
             </plugin>
         </gazebo>
+        <gazebo reference="front_right_wheel">
+            <surface>
+                <friction>
+                    <mu>0.7</mu>
+                    <mu2>0.0</mu2>
+                    <fdir1>1 0 0</fdir1>
+                    <slip1>1.0</slip1>
+                    <slip2>1.0</slip2>
+                </friction>
+            </surface>
+        </gazebo>
+        <gazebo reference="front_left_wheel">
+            <surface>
+                <friction>
+                    <mu>0.7</mu>
+                    <mu2>0.0</mu2>
+                    <fdir1>1 0 0</fdir1>
+                    <slip1>1.0</slip1>
+                    <slip2>1.0</slip2>
+                </friction>
+            </surface>
+        </gazebo>
+        <gazebo reference="rear_right_wheel">
+            <surface>
+                <friction>
+                    <mu>0.7</mu>
+                    <mu2>0.0</mu2>
+                    <fdir1>1 0 0</fdir1>
+                    <slip1>1.0</slip1>
+                    <slip2>1.0</slip2>
+                </friction>
+            </surface>
+        </gazebo>
+        <gazebo reference="rear_left_wheel">
+            <surface>
+                <friction>
+                    <mu>0.7</mu>
+                    <mu2>0.0</mu2>
+                    <fdir1>1 0 0</fdir1>
+                    <slip1>1.0</slip1>
+                    <slip2>1.0</slip2>
+                </friction>
+            </surface>
+        </gazebo>
     </xacro:macro>
 </robot>

Commit message: Static TF fix

File: scout_mini_description/models/scout_mini/xacro/scout_mini_tf.xacro (robot description, xacro)
@@ -42,5 +42,5 @@
             <mass value="60" />
             <origin xyz="0.0 0.0 0.0" />
-            <inertia ixx="2.288641" ixy="0" ixz="0" iyy="5.103976" iyz="0" izz="3.431465" />
+            <inertia ixx="3.0" ixy="0" ixz="0" iyy="2.5" iyz="0" izz="3.431465" />
         </inertial>
     </link>
@@ -52,5 +52,5 @@
     <link name="base_footprint" />
     <joint name="base_footprint_joint" type="fixed">
-        <origin xyz="0 0 -0.16" />
+        <origin xyz="0 0 0.16" />
         <parent link="base_footprint"/>
         <child link="base_link"/>

File: scout_mini_gazebo/models/scout_mini/xacro/scout_mini_sensors.xacro (robot description, xacro)
@@ -54,5 +54,5 @@
                 <update_rate>100</update_rate>
                 <visualize>true</visualize>
-                <!-- <imu>
+                <imu>
                     <angular_velocity>
                         <x>
@@ -107,5 +107,5 @@
                         </z>
                     </linear_acceleration>
-                </imu> -->
+                </imu>
             </sensor>
         </gazebo>
