Commit message: NAV2 configuration update

File: scout_mini_gazebo/models/scout_mini/xacro/scout_mini.xacro (robot description, xacro)
@@ -73,10 +73,10 @@
     <xacro:IMU />
     <xacro:depth_camera />
-    <link name="base_footprint" />
+    <!-- <link name="base_footprint" />
     <joint name="base_footprint_joint" type="fixed">
         <origin xyz="0 0 0.16" />
         <parent link="base_footprint" />
         <child link="base_link" />
-    </joint>
+    </joint> -->
     <link name="front_mount" />
     <joint name="front_mount_joint" type="fixed">

File: scout_mini_gazebo/models/scout_mini/xacro/scout_mini_gazebo.xacro (robot description, xacro)
@@ -32,5 +32,5 @@
                 <odometry_topic>zed_node/odom</odometry_topic>
                 <odometry_frame>odom</odometry_frame>
-                <robot_base_frame>base_footprint</robot_base_frame>
+                <robot_base_frame>base_link</robot_base_frame>
             </plugin>
         </gazebo>

File: scout_mini_gazebo/models/scout_mini/xacro/scout_mini_sensors.xacro (robot description, xacro)
@@ -13,10 +13,10 @@
         </xacro:zed_camera>
         <link name="zed_depth_link_optical" />
-        <joint name="zed_depth_join_optical" type="fixed">
+        <joint name="zed_depth_joint_optical" type="fixed">
             <parent link="zed_mount_link" />
             <child link="zed_depth_link_optical" />
             <origin xyz="0 0 0" rpy="${-pi/2} 0 ${-pi/2}" />
         </joint>
-        <gazebo reference="zed_mount_link">
+        <gazebo reference="zed2_camera_center">
             <sensor type="depth" name="zed_depth_camera">
                 <visualize>false</visualize>
@@ -42,5 +42,5 @@
                         <!-- Remappings for the ZED Camera Nodes -->
                     </ros>
-                    <frame_name>zed_depth_link_optical</frame_name>
+                    <frame_name>zed2_right_camera_optical_frame</frame_name>
                     <cameraName>zed_depth_camera</cameraName>
                     <hack_baseline>0.07</hack_baseline>

Commit message: EKF modifications

File: scout_mini_gazebo/models/scout_mini/xacro/scout_mini.xacro (robot description, xacro)
@@ -73,10 +73,10 @@
     <xacro:IMU />
     <xacro:depth_camera />
-    <!-- <link name="base_footprint" />
+    <link name="base_footprint" />
     <joint name="base_footprint_joint" type="fixed">
         <origin xyz="0 0 0.16" />
         <parent link="base_footprint" />
         <child link="base_link" />
-    </joint> -->
+    </joint>
     <link name="front_mount" />
     <joint name="front_mount_joint" type="fixed">

Commit message: Fixed Gazebo inertias

File: scout_mini_gazebo/models/scout_mini/xacro/scout_mini.xacro (robot description, xacro)
@@ -44,7 +44,7 @@
         <inertial>
             <mass value="60" />
-            <origin xyz="0.0 0.0 0.0" />
+            <origin xyz="0.0 0.0 0.05" />
             <!-- <inertia ixx="2.288641" ixy="0" ixz="0" iyy="5.103976" iyz="0" izz="3.431465" /> -->
-            <inertia ixx="3.0" ixy="0" ixz="0" iyy="3.0" iyz="0" izz="3.431465" />
+            <inertia ixx="3.0" ixy="0" ixz="0" iyy="2.5" iyz="0" izz="3.431465" />
         </inertial>
     </link>

Commit message: Fixed static TF

File: scout_mini_gazebo/models/scout_mini/xacro/scout_mini.xacro (robot description, xacro)
@@ -45,5 +45,4 @@
             <mass value="60" />
             <origin xyz="0.0 0.0 0.05" />
-            <!-- <inertia ixx="2.288641" ixy="0" ixz="0" iyy="5.103976" iyz="0" izz="3.431465" /> -->
             <inertia ixx="3.0" ixy="0" ixz="0" iyy="2.5" iyz="0" izz="3.431465" />
         </inertial>
