Commit message: DDS_XML

File: scout_mini_description/models/commander_slim/xacro/commander_slim.xacro (robot description, xacro)
@@ -24,7 +24,14 @@
     </link>
     <joint name="commander_slim_joint" type="fixed">
-        <origin xyz="0.0 0.0 0.05" rpy="0 0 0" />
+        <origin xyz="0.0 0.0 0.068" rpy="0 0 0" />
         <parent link="base_link" />
         <child link="commander_slim_link" />
+    </joint>
+    <link name="IMU">
+    </link>
+    <joint name="IMU_joint" type="fixed">
+        <origin xyz="0.12975 0.04175 0.123201" rpy="${pi} 0 ${pi/2}" />
+        <parent link="commander_slim_link" />
+        <child link="IMU" />
     </joint>
     <joint name="zed_mount_joint" type="fixed">

Commit message: Fixed viz - IMU Launch

File: scout_mini_description/models/commander_slim/xacro/commander_slim.xacro (robot description, xacro)
@@ -1,5 +1,4 @@
 <?xml version="1.0"?>
 <robot name="commander_slim" xmlns:xacro="http://www.ros.org/wiki/xacro">
-    <xacro:include filename="$(find zed_wrapper)/urdf/zed_macro.urdf.xacro" />
     <link name="commander_slim_link">
         <visual>
@@ -35,12 +34,3 @@
         <child link="IMU" />
     </joint>
-    <joint name="zed_mount_joint" type="fixed">
-        <origin xyz="0.277812 0 0.108212" rpy="0 0 0" />
-        <parent link="commander_slim_link" />
-        <child link="zed_mount_link" />
-    </joint>
-    <link name="zed_mount_link" />
-    <xacro:zed_camera name="zed2" model="zed2" parent="zed_mount_link">
-      <origin xyz="0 0 0" rpy="0 0 0" />
-    </xacro:zed_camera>
 </robot>

Commit message: Added microstrain sensor_wgs84 joint

File: scout_mini_description/models/commander_slim/xacro/commander_slim.xacro (robot description, xacro)
@@ -34,3 +34,9 @@
         <child link="IMU" />
     </joint>
+    <link name="sensor_wgs84"/>
+    <joint name="microstrain_joint" type="fixed">
+        <origin xyz="0.12975 0.04175 0.123201" rpy="${pi} 0 ${pi/2}" />
+        <parent link="commander_slim_link" />
+        <child link="sensor_wgs84" />
+    </joint>
 </robot>
